File: bus_vsens_on_off.kicad_sch (KiCad schematic)
At the start: 19 parts, among them J9 Conn_01x02, Q7 FMMT493TA, Q8 FMMT593TA

Commit message: some routing processing
Parts:
- added C58: 10uF, Capacitor_SMD:C_1206_3216Metric, symbol Device:C_Small
- added C59: 2.2uF, Capacitor_SMD:C_0402_1005Metric, symbol Device:C_Small
- added H1, H2, H3, H4: MountingHole, MountingHole:MountingHole_3.2mm_M3_ISO14580, symbol Mechanical:MountingHole
- added U5: LP5912-3.3DRV, Package_SON:WSON-6-1EP_2x2mm_P0.65mm_EP1x1.6mm_ThermalVias, symbol Regulator_Linear:LP5912-3.3DRV
- C53: footprint Capacitor_SMD:C_0603_1608Metric -> Capacitor_SMD:C_0402_1005Metric
- R39, R40, R41, R42, R43, R44, R45, R46, R47, R48, R49, R50, R51, R52, R53: footprint Resistor_SMD:R_0603_1608Metric -> Resistor_SMD:R_0402_1005Metric
Connections:
- net GND: now also C58.2, C59.2, U5.5 (GND), U5.7 (EP)
- net POWER_ON: now also U5.4 (EN)
- new net +15V: C58.1, U5.6 (IN)
- new net +3.3V: C59.1, U5.1 (OUT)
- no-connect marks 0 -> 1
