File: inverter.kicad_sch (KiCad schematic)
At the start: 41 parts, among them Q1 CSD19536KTT, Q2 CSD19536KTT, Q3 CSD19536KTT, Q4 CSD19536KTT, Q5 CSD19536KTT, Q6 CSD19536KTT, U4 INA180A3IDBVT

Commit message: some routing processing
Parts:
- added H5, H6, H7: MountingHole_Pad, MountingHole:MountingHole_2.2mm_M2_Pad_Via, symbol Mechanical:MountingHole_Pad
- C42, C44, C49: footprint Capacitor_SMD:C_0603_1608Metric -> Capacitor_SMD:C_0402_1005Metric
- R32, R33, R36: footprint Resistor_SMD:R_0603_1608Metric -> Resistor_SMD:R_0402_1005Metric
Connections:
- net SHA: now also H5.1
- net SHB: now also H6.1
- net SHC: now also H7.1
