File: mcu.kicad_sch (KiCad schematic)
At the start: 26 parts, among them J4 BOOT, J5 SWD, J6 USB_C, SW2 RESET, U2 STM32F103C8Tx, Y2 8Mhz

Commit message: schematic finished
Parts:
- added C1, C10, C13, C7: 100nF, Capacitor_SMD:C_0603_1608Metric, symbol Device:C_Small
- added C14, C15, C16: 1000pF, Capacitor_SMD:C_0603_1608Metric, symbol Device:C_Small
- added J2: Conn_01x02, Connector_PinHeader_2.54mm:PinHeader_1x02_P2.54mm_Vertical, symbol Connector_Generic:Conn_01x02
- added J5: HALL, Connector_PinSocket_2.54mm:PinSocket_1x05_P2.54mm_Vertical, symbol Connector_Generic:Conn_01x05
- added J6: Speed, Connector_PinHeader_2.54mm:PinHeader_1x04_P2.54mm_Vertical, symbol Connector_Generic:Conn_01x04
- added R11, R13, R9: 3.3k, Resistor_SMD:R_0603_1608Metric, symbol Device:R_Small
- added R12, R5: 10k, Resistor_SMD:R_0603_1608Metric, symbol Device:R_Small
- added R15: 1M, Resistor_SMD:R_0603_1608Metric, symbol Device:R_Small
- added R8: 2M, Resistor_SMD:R_0603_1608Metric, symbol Device:R_Small
- added U1: TMP235A4DBZR, Package_TO_SOT_SMD:SOT-23, symbol Regulator_Linear:APE8865N-24-HF-3
- D1: renamed from D4; footprint (none) -> LED_SMD:LED_0603_1608Metric
- D2: renamed from D5; footprint (none) -> LED_SMD:LED_0603_1608Metric
- renumbered C18 to C11, C17 to C12, C10 to C2, C11 to C3, C12 to C4, C13 to C5, C14 to C6, C16 to C8, C15 to C9, D6 to D3, J4 to J1, J5 to J3, J6 to J7, R9 to R1, R15 to R10, R16 to R14, R11 to R2, R13 to R3, R14 to R4, R12 to R6, R10 to R7, SW2 to SW1, Y2 to Y1
Connections:
- net +3.3V: now also C1.1, J5.5 (Pin_5), J6.3 (Pin_3), R11.2, R13.2, R8.2, R9.2, U1.3 (VI)
- net GND: now also C1.2, C10.2, C13.2, C14.2, C15.1, C16.1, C7.2, J2.2 (Pin_2), J5.4 (Pin_4), J6.1 (Pin_1), R15.1, U1.1 (GND)
- net LED: now also U2.41 (PB5); no longer U2.2 (PC13)
- net RESET: now also SW1.2 (B); no longer SW1.3 (B)
- net Speed_Ref: now reaches U2.10 (PA0)
- net Speed_Ref: now also C13.1, R12.2, R15.2
- net BEMF_A: now reaches U2.11 (PA1)
- net BEMF_A: now also U2.2 (PC13)
- net BEMF_B: now reaches U2.12 (PA2)
- net BEMF_B: now also U2.3 (PC14)
- net BEMF_C: now reaches U2.13 (PA3)
- net BEMF_C: now also U2.4 (PC15)
- net Temp_Sense: now reaches U2.14 (PA4)
- net Temp_Sense: now also C7.1, R5.2
- net IA_IDC: now reaches U2.15 (PA5)
- net INH_C: now reaches U2.16 (PA6)
- net INL_C: now reaches U2.17 (PA7)
- net FAULT: now reaches U2.18 (PB0)
- net HB: now reaches U2.21 (PB10)
- net HB: now also C15.2, J5.2 (Pin_2), R11.1
- net HC: now reaches U2.22 (PB11)
- net HC: now also C14.1, J5.3 (Pin_3), R9.1
- net SCS: now reaches U2.25 (PB12)
- net SCLK: now reaches U2.26 (PB13)
- net SDO: now reaches U2.27 (PB14)
- net SDI: now reaches U2.28 (PB15)
- net INL_A: now reaches U2.30 (PA9)
- net INH_A: now reaches U2.31 (PA10)
- net INH_B: now reaches U2.38 (PA15)
- net INL_B: now reaches U2.39 (PB3)
- net DIR: now reaches U2.42 (PB6)
- net DIR: now also C10.1, J2.1 (Pin_1), R8.1
- net DC_FB: now reaches U2.43 (PB7)
- net ENABLE_GD: now reaches U2.45 (PB8)
- net HA: now reaches U2.46 (PB9)
- net HA: now also C16.2, J5.1 (Pin_1), R13.1
- new net: R5.1, U1.2 (VO)
- new net: J6.2 (Pin_2), R12.1
- new net POWER_ON: J6.4 (Pin_4)
Other:
- note added: "Boot & Reset"
- note added: "Crystal"
- note added: "DIR"
- note added: "Decoupling Cap"
- note added: "HALL Conn"
- note added: "LED"
- note added: "MCU"
- note added: "SWD"
- note added: "Speed Ref"
- note added: "Temp Sense"
- note added: "USB-C"
- title: (none) -> MCU and Periphs
- moved on the sheet: C11, C12, C2, C3, C4, C5, C6, C8, C9, D1, D2, D3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

Commit message: some routing processing
Parts:
- removed C1, C10, C11, C13: 100nF, Capacitor_SMD:C_0603_1608Metric, symbol Device:C_Small
- added C54, C55, C56, C57: 100nF, Capacitor_SMD:C_0402_1005Metric, symbol Device:C_Small
- C14, C15, C16, C2, C3, C4, C5, C6, C7, C8, C9: footprint Capacitor_SMD:C_0603_1608Metric -> Capacitor_SMD:C_0402_1005Metric
- R1, R10, R11, R12, R13, R14, R15, R2, R3, R4, R5, R6, R7, R8, R9: footprint Resistor_SMD:R_0603_1608Metric -> Resistor_SMD:R_0402_1005Metric
Connections:
- net +3.3V: now also C7.1, C56.1
- net DIR: now also C55.1
- net GND: now also C15.2, C16.2, R14.1, C54.2, C55.2, C56.2, C57.2; no longer C15.1, C16.1, R14.2
- net HA: now also C16.1; no longer C16.2
- net HB: now also C15.1, U2.22 (PB11); no longer C15.2, U2.21 (PB10)
- net HC: now also U2.21 (PB10); no longer U2.22 (PB11)
- net INH_C: now also U2.17 (PA7); no longer U2.16 (PA6)
- net INL_C: now also U2.16 (PA6); no longer U2.17 (PA7)
- net Speed_Ref: now also C57.1
- net Temp_Sense: now also C54.1; no longer C7.1
- net at J7.B5 (CC2): now also R14.2; no longer R14.1
