File: BLDC Motor Driver.kicad_pcb (KiCad board)
At the start: 2 copper layers, 139 parts, among them J1 BOOT, J2 Conn_01x02, J3 SWD, J4 Conn_01x02, J5 HALL, J6 Speed, J7 USB_C, J8 Conn_01x02, J9 Conn_01x02, Q1 CSD19536KTT, Q2 CSD19536KTT, Q3 CSD19536KTT, Q4 CSD19536KTT, Q5 CSD19536KTT, Q6 CSD19536KTT, Q7 FMMT493TA, Q8 FMMT593TA, SW1 RESET, U1 TMP235A4DBZR, U2 STM32F103C8Tx, U3 DRV8350RHRGZT, U4 INA180A3IDBVT, Y1 8Mhz

Commit message: some routing processing
Parts:
- removed C1, C10, C11, C13: 100nF, Capacitor_SMD:C_0603_1608Metric
- removed J4: Conn_01x02, Connector_PinHeader_2.54mm:PinHeader_1x02_P2.54mm_Vertical
- added C54: 100nF, Capacitor_SMD:C_0402_1005Metric, B.Cu at (183.8, 102.6)
- added C55: 100nF, Capacitor_SMD:C_0402_1005Metric, F.Cu at (172.9, 106.2)
- added C56: 100nF, Capacitor_SMD:C_0402_1005Metric, F.Cu at (197.4, 96.8)
- added C57: 100nF, Capacitor_SMD:C_0402_1005Metric, F.Cu at (196.1, 58.9)
- added C58: 10uF, Capacitor_SMD:C_1206_3216Metric, F.Cu at (161.5, 55.2)
- added C59: 2.2uF, Capacitor_SMD:C_0402_1005Metric, F.Cu at (164.4, 58.0)
- added H1: MountingHole, MountingHole:MountingHole_3.2mm_M3_ISO14580, F.Cu at (106.0, 45.1)
- added H2: MountingHole, MountingHole:MountingHole_3.2mm_M3_ISO14580, F.Cu at (196.8, 45.1)
- added H3: MountingHole, MountingHole:MountingHole_3.2mm_M3_ISO14580, F.Cu at (160.8, 81.1)
- added H4: MountingHole, MountingHole:MountingHole_3.2mm_M3_ISO14580, F.Cu at (106.0, 107.0)
- added H5: MountingHole_Pad, MountingHole:MountingHole_2.2mm_M2_Pad_Via, F.Cu at (129.3, 54.3)
- added H6: MountingHole_Pad, MountingHole:MountingHole_2.2mm_M2_Pad_Via, F.Cu at (129.0, 69.0)
- added H7: MountingHole_Pad, MountingHole:MountingHole_2.2mm_M2_Pad_Via, F.Cu at (129.0, 86.0)
- added U5: LP5912-3.3DRV, Package_SON:WSON-6-1EP_2x2mm_P0.65mm_EP1x1.6mm_ThermalVias, F.Cu at (164.0, 56.2)
- C14, C15, C16, C2, C20, C23, C25, C26, C3, C4, C42, C44, C49, C5, C53, C6, C8, C9: footprint Capacitor_SMD:C_0603_1608Metric -> Capacitor_SMD:C_0402_1005Metric
- C24: footprint Capacitor_SMD:C_0603_1608Metric -> Capacitor_SMD:C_0805_2012Metric
- C27: footprint Capacitor_SMD:C_0603_1608Metric -> Capacitor_SMD:C_0402_1005Metric; moved to F.Cu
- C28, C29, C30, D6, D7, L2: moved to F.Cu
- C35, C45, C52, R30, R31, U1: moved to B.Cu
- C7: footprint Capacitor_SMD:C_0603_1608Metric -> Capacitor_SMD:C_0402_1005Metric; moved to B.Cu
- R1, R10, R11, R12, R13, R14, R15, R16, R17, R18, R19, R2, R20, R3, R32, R33, R36, R39, R4, R40, R41, R42, R43, R44, R48, R49, R50, R51, R52, R53, R6, R7, R8, R9: footprint Resistor_SMD:R_0603_1608Metric -> Resistor_SMD:R_0402_1005Metric
- R21, R22, R23, R24, R25, R26, R27: footprint Resistor_SMD:R_0603_1608Metric -> Resistor_SMD:R_0402_1005Metric; moved to F.Cu
- R45, R46, R47, R5: footprint Resistor_SMD:R_0603_1608Metric -> Resistor_SMD:R_0402_1005Metric; moved to B.Cu
- moved C35 118.1 mm to (128.7, 49.3), turned to 0 degrees
- moved D8 105.0 mm to (115.9, 94.8), turned to 180 degrees
- moved C47 98.2 mm to (125.2, 88.5), turned to 90 degrees
- moved C31 98.2 mm to (125.0, 55.9), turned to 90 degrees
- moved C36 98.2 mm to (125.2, 71.5), turned to 90 degrees
- moved C37 97.1 mm to (152.1, 71.4)
- moved C32 97.1 mm to (151.9, 55.7)
- moved C33 97.1 mm to (125.3, 46.6)
- moved C34 97.1 mm to (130.2, 46.6)
- moved C40 97.1 mm to (125.5, 62.3)
- moved C41 97.1 mm to (130.7, 62.3)
- moved C43 97.1 mm to (153.4, 103.5)
- moved C46 97.1 mm to (155.8, 103.5)
- moved C48 97.1 mm to (151.9, 88.3)
- moved C50 97.1 mm to (125.1, 79.1)
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Connections:
- C15 pad 1: GND -> HB
- C15 pad 2: HB -> GND
- C16 pad 1: GND -> HA
- C16 pad 2: HA -> GND
- C7 pad 1: Temp_Sense -> +3.3V
- R14 pad 1: Net-(J7-CC2) -> GND
- R14 pad 2: GND -> Net-(J7-CC2)
- U2 pad 16: INH_C -> INL_C
- U2 pad 17: INL_C -> INH_C
- U2 pad 21: HB -> HC
- U2 pad 22: HC -> HB
Routing:
- net GHC: track 0.00 -> 71.6 mm, vias 0 -> 2
- net SLA: track 0.00 -> 63.5 mm, vias 0 -> 50
- net SHA: track 0.00 -> 63.1 mm, vias 0 -> 19
- net GHA: track 0.00 -> 55.1 mm, vias 0 -> 2
- net GHB: track 0.00 -> 53.8 mm, vias 0 -> 2
- net INL_C: track 0.00 -> 52.5 mm, vias 0 -> 2
- net INH_C: track 0.00 -> 48.7 mm, vias 0 -> 2
- net HA: track 0.00 -> 46.3 mm, vias 0 -> 2
- net INH_A: track 0.00 -> 36.8 mm, vias 0 -> 2
- net INL_A: track 0.00 -> 35.3 mm, vias 0 -> 2
- net INH_B: track 0.00 -> 30.9 mm, vias 0 -> 2
- net INL_B: track 0.00 -> 29.2 mm, vias 0 -> 2
- net /STM32F103 MCU/SWDCLK: track 0.00 -> 28.4 mm
- net ENABLE_GD: track 0.00 -> 26.5 mm
- net GLA: track 0.00 -> 26.3 mm, vias 0 -> 2
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- added copper zone on In2.Cu, net +15V
- added copper zone on In2.Cu, net +3.3V
- added copper zone on F.Cu, net +5VDC
- added copper zone on B.Cu, net GND
- added copper zone on F.Cu, net GND
- added copper zone on F.Cu, net Net-(D3-A)
- added copper zone on F.Cu, net SHA
- added copper zone on F.Cu, net SHB
- added copper zone on F.Cu, net SHC
- added copper zone on F.Cu, net SLA
- added copper zone on F.Cu, net VDC
- added copper zone on In2.Cu, net VDC
- added copper zone on In2.Cu, net VGD
Other:
- board outline added: 101 x 72 mm
- copper layers 2 -> 4

Commit message: finished the pcb design
Parts:
- Y1: footprint Crystal:Crystal_HC18-U_Vertical -> Crystal:Crystal_HC49-4H_Vertical
- moved R16 14.5 mm to (167.4, 71.1), turned to 0 degrees
- moved D4 14.0 mm to (166.9, 72.4)
- moved D2 13.3 mm to (156.5, 76.0), turned to 0 degrees
- moved R4 10.6 mm to (156.2, 74.6), turned to 0 degrees
- moved R19 2.68 mm to (167.4, 73.9), turned to 180 degrees
- moved C5 0.93 mm to (181.8, 99.4), turned to 0 degrees
- moved C6 0.70 mm to (174.8, 86.5)
- moved R30 0.57 mm to (173.4, 98.9)
- moved R31 0.56 mm to (169.5, 98.9)
- moved J1 0.42 mm to (176.2, 76.7)
- moved R45 0.40 mm to (171.4, 92.9)
- moved R46 0.40 mm to (171.4, 91.9)
- moved R47 0.40 mm to (171.4, 91.0)
- moved C49 0.30 mm to (166.3, 105.4)
- moved C55 0.30 mm to (173.0, 106.5)
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Routing:
- net SHB: track 0.00 -> 76.1 mm, vias 13 -> 17
- net SHC: track 3.46 -> 74.2 mm, vias 14 -> 18
- net VGD: track 12.4 -> 80.1 mm, vias 0 -> 2
- net SDI: track 5.26 -> 66.1 mm, vias 0 -> 4
- net SCS: track 3.03 -> 61.4 mm, vias 0 -> 4
- net POWER_ON: track 0.00 -> 58.3 mm
- net Speed_Ref: track 7.79 -> 65.8 mm, vias 2 -> 4
- net SDO: track 6.66 -> 62.7 mm, vias 0 -> 4
- net /STM32F103 MCU/RESET: track 8.60 -> 64.1 mm, vias 0 -> 6
- net /STM32F103 MCU/BOOT1: track 0.00 -> 54.1 mm, vias 0 -> 2
- net SCLK: track 5.78 -> 54.7 mm, vias 0 -> 4
- net FAULT: track 5.56 -> 54.0 mm, vias 1 -> 4
- net VDC: track 20.2 -> 60.7 mm, vias 140 -> 142
- net SLA: track 63.5 -> 103.5 mm, vias 50 -> 51
- net GND: track 0.21 -> 36.4 mm, vias 19 -> 53
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- added copper zone on F.Cu, net +15V
- added copper zone on F.Cu, net +3.3V
- added copper zone on In1.Cu, net GND
- added copper zone on In2.Cu, net SLA
- added copper zone on B.Cu, net VDC
